File: SolderChallenge.sch (KiCad schematic (older format))
At the start: 33 parts, among them Q1 MOS_N, Q2 MOS_N, Q3 MOS_N, Q4 MOS_N_x2, U1 555, U2 555, U3 555

Commit message: Modified Q1 to use wide variant of package as that's what I ordred. RS had wrong info on site.
Parts:
- Q1: footprint SolderChallenge:TO-92_Inline_Narrow_Oval_SGD -> SolderChallenge:TO-92_Inline_Wide_SGD
Changed lines of the file:
@@
 F 0 "Q1" H 4260 2270 50  0000 R CNN
 F 1 "MOS_N" H 4200 1950 50  0000 R CNN
-F 2 "SolderChallenge:TO-92_Inline_Narrow_Oval_SGD" H 4250 2100 60  0001 C CNN
+F 2 "SolderChallenge:TO-92_Inline_Wide_SGD" H 4250 2100 60  0001 C CNN
 F 3 "" H 4250 2100 60  0000 C CNN
 	1    4250 2100

Commit message: Update to KiCAD v5.0
Parts:
- BT1: symbol Battery -> SolderChallenge:Battery
- C1, C2, C3: symbol C -> SolderChallenge:C
- D1: symbol DIODE -> SolderChallenge:DIODE
- LED1, LED2, LED3, LED4, LED5: symbol LED -> SolderChallenge:LED
- Q1, Q2, Q3: symbol MOS_N -> SolderChallenge:MOS_N
- Q4: symbol MOS_N_x2 -> SolderChallenge:MOS_N_x2
- R1, R10, R11, R12, R13, R14, R15, R16, R2, R3, R4, R5, R6, R7, R8, R9: symbol R -> SolderChallenge:R
- U1, U2, U3: symbol LM555N -> SolderChallenge:LM555N
Connections:
- net +9V: now also D1.A; no longer D1.1 (A)
- net VCC: now also D1.C; no longer D1.2 (K)

Commit message: Forgot to update schematic footprints when I changed them in the layout. I wish KiCAD would automatically back-annotate, or at least let you choose to
Parts:
- C1: footprint SolderChallenge:CP_Radial_D5.0mm_P2.00mm -> SolderChallenge:C_Disc_D5.1mm_W3.2mm_P5.00mm
- Q3: footprint SolderChallenge:SOT-323_SC-70_GSD_Handsoldering -> SolderChallenge:SOT-23_GSD_Nexperia_TO-236AB
Changed lines of the file:
@@
 F 0 "C1" H 6675 3000 50  0000 L CNN
 F 1 "2.2u" H 6675 2800 50  0000 L CNN
-F 2 "SolderChallenge:CP_Radial_D5.0mm_P2.00mm" H 6688 2750 50  0001 C CNN
+F 2 "SolderChallenge:C_Disc_D5.1mm_W3.2mm_P5.00mm" H 6688 2750 50  0001 C CNN
 F 3 "" H 6650 2900 50  0001 C CNN
 	1    6650 2900
@@
 F 0 "Q3" H 10610 2220 50  0000 R CNN
 F 1 "MOS_N" H 10550 1900 50  0000 R CNN
-F 2 "SolderChallenge:SOT-323_SC-70_GSD_Handsoldering" H 10600 2050 60  0001 C CNN
+F 2 "SolderChallenge:SOT-23_GSD_Nexperia_TO-236AB" H 10600 2050 60  0001 C CNN
 F 3 "" H 10600 2050 60  0000 C CNN
 	1    10600 2050

Commit message: Increase pin spacing on R1-5. Originally used 7.68mm. Increase to 9mm to make insertion easier
Parts:
- R1, R2, R3, R4, R5: footprint SolderChallenge:R_Axial_DIN0207_L6.3mm_D2.5mm_P7.62mm_Horizontal -> SolderChallenge:R_Axial_DIN0207_L6.3mm_D2.5mm_P9.00mm_Horizontal
Changed lines of the file:
@@
 F 0 "R2" V 2230 1600 50  0000 C CNN
 F 1 "390" V 2150 1600 50  0000 C CNN
-F 2 "SolderChallenge:R_Axial_DIN0207_L6.3mm_D2.5mm_P7.62mm_Horizontal" V 2080 1600 50  0001 C CNN
+F 2 "SolderChallenge:R_Axial_DIN0207_L6.3mm_D2.5mm_P9.00mm_Horizontal" V 2080 1600 50  0001 C CNN
 F 3 "" H 2150 1600 50  0001 C CNN
 	1    2150 1600
@@
 F 0 "R3" V 2430 1600 50  0000 C CNN
 F 1 "390" V 2350 1600 50  0000 C CNN
-F 2 "SolderChallenge:R_Axial_DIN0207_L6.3mm_D2.5mm_P7.62mm_Horizontal" V 2280 1600 50  0001 C CNN
+F 2 "SolderChallenge:R_Axial_DIN0207_L6.3mm_D2.5mm_P9.00mm_Horizontal" V 2280 1600 50  0001 C CNN
 F 3 "" H 2350 1600 50  0001 C CNN
 	1    2350 1600
@@
 F 0 "R4" V 2630 1600 50  0000 C CNN
 F 1 "390" V 2550 1600 50  0000 C CNN
-F 2 "SolderChallenge:R_Axial_DIN0207_L6.3mm_D2.5mm_P7.62mm_Horizontal" V 2480 1600 50  0001 C CNN
+F 2 "SolderChallenge:R_Axial_DIN0207_L6.3mm_D2.5mm_P9.00mm_Horizontal" V 2480 1600 50  0001 C CNN
 F 3 "" H 2550 1600 50  0001 C CNN
 	1    2550 1600
@@
 F 0 "R1" V 2030 1600 50  0000 C CNN
 F 1 "390" V 1950 1600 50  0000 C CNN
-F 2 "SolderChallenge:R_Axial_DIN0207_L6.3mm_D2.5mm_P7.62mm_Horizontal" V 1880 1600 50  0001 C CNN
+F 2 "SolderChallenge:R_Axial_DIN0207_L6.3mm_D2.5mm_P9.00mm_Horizontal" V 1880 1600 50  0001 C CNN
 F 3 "" H 1950 1600 50  0001 C CNN
 	1    1950 1600
@@
 F 0 "R5" V 2830 1600 50  0000 C CNN
 F 1 "390" V 2750 1600 50  0000 C CNN
-F 2 "SolderChallenge:R_Axial_DIN0207_L6.3mm_D2.5mm_P7.62mm_Horizontal" V 2680 1600 50  0001 C CNN
+F 2 "SolderChallenge:R_Axial_DIN0207_L6.3mm_D2.5mm_P9.00mm_Horizontal" V 2680 1600 50  0001 C CNN
 F 3 "" H 2750 1600 50  0001 C CNN
 	1    2750 1600
